File: kicad/safeduino_mega_328.sch (KiCad schematic (older format))
At the start: 91 parts, among them X1 USB

Commit message: Начал разрабатывать принципиальную схему.
Parts:
- removed C21: 22мк 10В, symbol CAPITORS_ELECTROLYTIC
- removed C23: 0.1мк, symbol CAPITORS
- removed C7: 47мк 10В, symbol CAPITORS_ELECTROLYTIC
- removed DA3: LM1117DTX-3.3, symbol LM1117
- removed FU2: MF-MSMF050, ~, symbol PROTECTOR
- removed R1: 20к, symbol RESISTOR_TRIMMING
- removed R5: 1к, symbol RESISTOR
- removed VD1, VD2: SS14, symbol SHOTTKY_DIODE
- removed VT1: MMBT5551, symbol NPN
- removed XP3: DG126-5.0-02P-14, ~, symbol PIN_M_2
- removed XP39, XP40: ~, ~, symbol PIN_M_1
- removed XP4: IDC-16MS, ~, symbol PIN_M_16
- removed XP5: PLS-3, ~, symbol PIN_M_3
- added C?: 0.1мк, symbol CAPITORS
- added DD4: MAX485_DIP_SO, ~, symbol MAX485_DIP_SO
- added R?: 120, symbol RESISTOR
Connections:
- net labels added: RS485A, RS485B
- net labels removed: VCCUSB
- wire segments 284 -> 256
Other:
- note removed: "+5V"
- note removed: "DB0"
- note removed: "DB1"
- note removed: "DB2"
- note removed: "DB3"
- note removed: "DB4"
- note removed: "DB5"
- note removed: "DB6"
- note removed: "DB7"
- note removed: "E"
- note removed: "LED"
- note removed: "LEDA"
- note removed: "LEDK"
- note removed: "R/W"
- note removed: "RS"
- note removed: "VCC"
- note removed: "VEE"
- moved on the sheet: C6, DA1
